File: Aurora_blueprint_1.kicad_sch (KiCad schematic)
At the start: 20 parts, among them J1 Raspberry_Pi_4, K1 Fujitsu_FTR-LYCA005x, K2 Fujitsu_FTR-LYCA005x, K3 Fujitsu_FTR-LYCA005x, K4 Fujitsu_FTR-LYCA005x, M1 Motor_DC, M2 Motor_DC, M3 Motor_DC, M4 Motor_DC, U1 LM2576HVS-5, U2 LM2576HVS-12

Commit message: implemented UART ping-pong communication with Raspberry pi
Parts:
- A1: value Arduino_UNO_R2 -> Arduino_UNO_R3
Changed lines of the file:
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@@
 		(comment 1 "- @lynet_101")
 		(comment 2 "- Sebastian_lindau-skands")
+		(comment 3 "if more power neeeded, the motor assembly can be powered parallel instead")
+		(comment 4 "if parallel motors, then additional 12v regulators might be needed")
 	)
 	(junction
@@
 			)
 		)
-		(property "Value" "Arduino_UNO_R2"
+		(property "Value" "Arduino_UNO_R3"
 			(at 163.83 33.9246 90)
 			(effects

Commit message: Updated circuit schematics to align with IRL wirrering
Connections:
- net at J1.10 (GPIO15/UART_RXD): now also A1.18 (D3); no longer A1.16 (D1/TX)
- net at J1.13 (GPIO27/SDIO_DAT3): no longer TP4.1
- net at J1.18 (GPIO24/SDIO_DAT0): no longer TP7.1
- net at J1.22 (GPIO25/SDIO_DAT1): no longer TP6.1
- net at J1.31 (GPCLK2/GPIO06): now also TP4.1
- net at J1.33 (GPIO13/PWM1): now also TP5.1
- net at J1.35 (GPIO19/SPI1_MISO/PCM_FS): now also TP6.1
- net at J1.37 (GPIO26/SDIO_DAT2): now also TP7.1; no longer TP5.1
- net at J1.8 (GPIO14/UART_TXD): now also A1.17 (D2); no longer A1.15 (D0/RX)
Changed lines of the file:
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@@
-	(wire
-		(pts
-			(xy 171.45 147.32) (xy 171.45 93.98)
-		)
-		(stroke
-			(width 0)
-			(type default)
-			(color 42 84 255 1)
-		)
-	)
 	(wire
 		(pts
@@
 	(wire
 		(pts
-			(xy 191.77 66.04) (xy 195.58 66.04)
-		)
-		(stroke
-			(width 0)
-			(type default)
-			(color 173 101 255 1)
+			(xy 181.61 147.32) (xy 181.61 78.74)
+		)
+		(stroke
+			(width 0)
+			(type default)
+			(color 0 0 0 1)
 		)
 	)
@@
 	(wire
 		(pts
-			(xy 171.45 93.98) (xy 195.58 93.98)
-		)
-		(stroke
-			(width 0)
-			(type default)
-			(color 42 84 255 1)
-		)
-	)
-	(wire
-		(pts
 			(xy 104.14 138.43) (xy 90.17 138.43)
 		)
@@
 	(wire
 		(pts
-			(xy 191.77 62.23) (xy 191.77 66.04)
-		)
-		(stroke
-			(width 0)
-			(type default)
-			(color 173 101 255 1)
+			(xy 201.93 147.32) (xy 201.93 116.84)
+		)
+		(stroke
+			(width 0)
+			(type default)
+			(color 65 78 255 1)
+		)
+	)
+	(wire
+		(pts
+			(xy 119.38 63.5) (xy 119.38 52.07)
+		)
+		(stroke
+			(width 0)
+			(type default)
+			(color 154 24 255 1)
 		)
 	)
@@
 	(wire
 		(pts
-			(xy 181.61 96.52) (xy 181.61 147.32)
-		)
-		(stroke
-			(width 0)
-			(type default)
-			(color 42 84 255 1)
+			(xy 201.93 116.84) (xy 264.16 116.84)
+		)
+		(stroke
+			(width 0)
+			(type default)
+			(color 65 78 255 1)
 		)
 	)
@@
 	(wire
 		(pts
+			(xy 264.16 83.82) (xy 261.62 83.82)
+		)
+		(stroke
+			(width 0)
+			(type default)
+		)
+	)
+	(wire
+		(pts
 			(xy 114.3 173.99) (xy 114.3 167.64)
 		)
@@
 	(wire
 		(pts
+			(xy 195.58 66.04) (xy 195.58 64.77)
+		)
+		(stroke
+			(width 0)
+			(type default)
+		)
+	)
+	(wire
+		(pts
 			(xy 44.45 105.41) (xy 44.45 71.12)
 		)
@@
 	(wire
 		(pts
+			(xy 195.58 63.5) (xy 119.38 63.5)
+		)
+		(stroke
+			(width 0)
+			(type default)
+			(color 154 24 255 1)
+		)
+	)
+	(wire
+		(pts
 			(xy 44.45 105.41) (xy 41.91 105.41)
 		)
@@
 	(wire
 		(pts
-			(xy 195.58 96.52) (xy 181.61 96.52)
-		)
-		(stroke
-			(width 0)
-			(type default)
-			(color 42 84 255 1)
+			(xy 264.16 116.84) (xy 264.16 83.82)
+		)
+		(stroke
+			(width 0)
+			(type default)
+			(color 65 78 255 1)
 		)
 	)
@@
 	(wire
 		(pts
-			(xy 116.84 52.07) (xy 116.84 62.23)
-		)
-		(stroke
-			(width 0)
-			(type default)
-			(color 173 101 255 1)
-		)
-	)
-	(wire
-		(pts
 			(xy 97.79 102.87) (xy 97.79 78.74)
 		)
@@
 	(wire
 		(pts
+			(xy 191.77 58.42) (xy 191.77 147.32)
+		)
+		(stroke
+			(width 0)
+			(type default)
+			(color 153 107 0 1)
+		)
+	)
+	(wire
+		(pts
 			(xy 88.9 115.57) (xy 88.9 58.42)
 		)
@@
 	(wire
 		(pts
+			(xy 181.61 78.74) (xy 195.58 78.74)
+		)
+		(stroke
+			(width 0)
+			(type default)
+			(color 0 0 0 1)
+		)
+	)
+	(wire
+		(pts
 			(xy 97.79 147.32) (xy 97.79 125.73)
 		)
@@
 	(wire
 		(pts
+			(xy 195.58 58.42) (xy 191.77 58.42)
+		)
+		(stroke
+			(width 0)
+			(type default)
+			(color 153 107 0 1)
+		)
+	)
+	(wire
+		(pts
 			(xy 97.79 102.87) (xy 104.14 102.87)
 		)
@@
 	(wire
 		(pts
-			(xy 114.3 63.5) (xy 114.3 52.07)
-		)
-		(stroke
-			(width 0)
-			(type default)
-			(color 173 101 255 1)
-		)
-	)
-	(wire
-		(pts
 			(xy 90.17 57.15) (xy 142.24 57.15)
 		)
@@
 	(wire
 		(pts
-			(xy 191.77 147.32) (xy 191.77 99.06)
-		)
-		(stroke
-			(width 0)
-			(type default)
-			(color 42 84 255 1)
-		)
-	)
-	(wire
-		(pts
 			(xy 87.63 59.69) (xy 87.63 91.44)
 		)
@@
 	(wire
 		(pts
-			(xy 116.84 62.23) (xy 191.77 62.23)
-		)
-		(stroke
-			(width 0)
-			(type default)
-			(color 173 101 255 1)
+			(xy 121.92 64.77) (xy 121.92 52.07)
+		)
+		(stroke
+			(width 0)
+			(type default)
+			(color 154 24 255 1)
 		)
 	)
@@
 	(wire
 		(pts
+			(xy 171.45 99.06) (xy 171.45 147.32)
+		)
+		(stroke
+			(width 0)
+			(type default)
+			(color 255 143 23 1)
+		)
+	)
+	(wire
+		(pts
 			(xy 104.14 115.57) (xy 88.9 115.57)
 		)
@@
 	(wire
 		(pts
+			(xy 195.58 99.06) (xy 171.45 99.06)
+		)
+		(stroke
+			(width 0)
+			(type default)
+			(color 255 143 23 1)
+		)
+	)
+	(wire
+		(pts
 			(xy 139.7 52.07) (xy 139.7 55.88)
 		)
@@
 	(wire
 		(pts
-			(xy 195.58 147.32) (xy 201.93 147.32)
-		)
-		(stroke
-			(width 0)
-			(type default)
-			(color 42 84 255 1)
-		)
-	)
-	(wire
-		(pts
 			(xy 86.36 173.99) (xy 86.36 161.29)
 		)
@@
 	(wire
 		(pts
-			(xy 195.58 101.6) (xy 195.58 147.32)
-		)
-		(stroke
-			(width 0)
-			(type default)
-			(color 42 84 255 1)
+			(xy 195.58 64.77) (xy 121.92 64.77)
+		)
+		(stroke
+			(width 0)
+			(type default)
+			(color 154 24 255 1)
 		)
 	)
@@
 		)
 	)
-	(wire
-		(pts
-			(xy 191.77 99.06) (xy 195.58 99.06)
-		)
-		(stroke
-			(width 0)
-			(type default)
-			(color 42 84 255 1)
-		)
-	)
-	(wire
-		(pts
-			(xy 195.58 63.5) (xy 114.3 63.5)
-		)
-		(stroke
-			(width 0)
-			(type default)
-			(color 173 101 255 1)
-		)
-	)
